File: uLI-04.brd (EAGLE design)
At the start: 57 x 38.5 mm, 40 parts, among them IC1 PIC18F14K50-I/SS, IC2 ADM2483, IC3 MCP130T, IC4 78L05F, J1 PICPROG2-V, J5 WEBP6, J6 WEBP6, J7 WEBP6, Q1 12.00 MHz, T1 IRF7306, X1 MINI-USB_SHIELD4P-USB-SPEC, X2 ARK1550/2_S

Commit message: Change value of LED resistors based on reality.
Parts:
- R11: value 10k -> 2k2
- R8: value 10k -> 100k
Changed lines of the file:
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@@
 <?xml version="1.0" encoding="utf-8"?>
 <!DOCTYPE eagle SYSTEM "eagle.dtd">
-<eagle version="7.2.0">
+<eagle version="9.2.2">
 <drawing>
 <settings>
-<setting alwaysvectorfont="yes"/>
+<setting alwaysvectorfont="no"/>
+<setting keepoldvectorfont="yes"/>
 <setting verticaltext="up"/>
 </settings>
@@
 <variantdefs>
 <variantdef name="master"/>
-<variantdef name="slave" current="yes"/>
+<variantdef name="slave"/>
 </variantdefs>
 <classes>
@@
 <param name="dpMaxLengthDifference" value="10mm"/>
 <param name="dpGapFactor" value="2.5"/>
-<param name="checkGrid" value="0"/>
 <param name="checkAngle" value="0"/>
 <param name="checkFont" value="1"/>
 <param name="checkRestrict" value="1"/>
+<param name="checkStop" value="0"/>
+<param name="checkValues" value="0"/>
+<param name="checkNames" value="1"/>
+<param name="checkWireStubs" value="1"/>
+<param name="checkPolygonWidth" value="0"/>
 <param name="useDiameter" value="31"/>
 <param name="maxErrors" value="50"/>
@@
 <attribute name="VALUE" x="14.2525" y="16.5375" size="1.27" layer="28" font="vector" ratio="15" rot="MR0"/>
 </element>
-<element name="OK1" library="optocoupler" package="DIL04" value="PC817" x="30.7975" y="31.115" populate="no" smashed="yes" rot="R90">
+<element name="OK1" library="optocoupler" package="DIL04" value="PC817" x="30.7975" y="31.115" smashed="yes" rot="R90">
+<attribute name="NAME" x="30.7975" y="33.194" size="1.27" layer="25" ratio="15" rot="R180" align="bottom-center"/>
 <attribute name="VALUE" x="30.7975" y="33.306" size="1.27" layer="27" ratio="15" rot="R180" align="bottom-center"/>
-<attribute name="NAME" x="30.7975" y="33.194" size="1.27" layer="25" ratio="15" rot="R180" align="bottom-center"/>
-</element>
-<element name="R1" library="rcl" package="R1206" value="1k" x="38.735" y="31.4325" populate="no" smashed="yes" rot="R90">
+</element>
+<element name="R1" library="rcl" package="R1206" value="1k" x="38.735" y="31.4325" smashed="yes" rot="R90">
 <attribute name="NAME" x="37.7825" y="33.9725" size="1.27" layer="25" font="vector" ratio="15"/>
 <attribute name="VALUE" x="39.9375" y="28.775" size="1.27" layer="27" font="vector" ratio="15" rot="R180"/>
 </element>
-<element name="R2" library="rcl" package="R1206" value="100k" x="21.59" y="20.955" populate="no" smashed="yes" rot="R270">
+<element name="R2" library="rcl" package="R1206" value="100k" x="21.59" y="20.955" smashed="yes" rot="R270">
 <attribute name="NAME" x="20.32" y="21.59" size="1.27" layer="25" font="vector" ratio="15" rot="R180"/>
 <attribute name="VALUE" x="19.05" y="22.225" size="1.27" layer="27" font="vector" ratio="15" rot="R270"/>
@@
 <attribute name="NAME" x="10.8425" y="33.02" size="1.27" layer="25" font="vector" ratio="15" rot="R180" align="bottom-center"/>
 </element>
-<element name="LED4" library="led" package="LED3MM" value="BLUE 2mA" x="54.9275" y="30.1625" populate="no" smashed="yes" rot="MR180">
+<element name="LED4" library="led" package="LED3MM" value="BLUE 2mA" x="54.9275" y="30.1625" smashed="yes" rot="MR180">
 <attribute name="NAME" x="57.06" y="30.4275" size="1.27" layer="26" ratio="15" rot="MR90" align="bottom-center"/>
 <attribute name="VALUE" x="57.5275" y="30.4275" size="1.27" layer="28" ratio="15" rot="MR90" align="bottom-center"/>
 </element>
-<element name="R8" library="rcl" package="R1206" value="10k" x="48.26" y="34.6075" populate="no" smashed="yes" rot="MR0">
+<element name="R8" library="rcl" package="R1206" value="100k" x="48.26" y="34.6075" smashed="yes" rot="MR0">
 <attribute name="NAME" x="49.23" y="36.095" size="1.27" layer="26" font="vector" ratio="15" rot="MR0"/>
 <attribute name="VALUE" x="49.53" y="36.0675" size="1.27" layer="28" font="vector" ratio="15" rot="MR0"/>
@@
 <attribute name="VALUE" x="30.7975" y="16.575" size="1.27" layer="28" font="vector" ratio="15" rot="MR180" align="top-center"/>
 </element>
-<element name="D2" library="diode" package="SMB" value="S2M" x="43.18" y="32.25" populate="no" smashed="yes" rot="MR90">
+<element name="D2" library="diode" package="SMB" value="S2M" x="43.18" y="32.25" smashed="yes" rot="MR90">
 <attribute name="NAME" x="40.961" y="33.509" size="1.27" layer="26" font="vector" ratio="15" rot="MR270"/>
 <attribute name="VALUE" x="39.751" y="31.091" size="1.27" layer="28" font="vector" ratio="15" rot="MR90"/>
 </element>
-<element name="OK2" library="optocoupler" package="DIL04" value="PC817" x="30.7975" y="36.83" populate="no" smashed="yes" rot="R270">
+<element name="OK2" library="optocoupler" package="DIL04" value="PC817" x="30.7975" y="36.83" smashed="yes" rot="R270">
+<attribute name="NAME" x="30.7975" y="34.751" size="1.27" layer="25" ratio="15" align="bottom-center"/>
 <attribute name="VALUE" x="30.7975" y="34.639" size="1.27" layer="27" ratio="15" align="bottom-center"/>
-<attribute name="NAME" x="30.7975" y="34.751" size="1.27" layer="25" ratio="15" align="bottom-center"/>
-</element>
-<element name="R9" library="rcl" package="R1206" value="1k" x="26.3525" y="26.3525" populate="no" smashed="yes" rot="R270">
+</element>
+<element name="R9" library="rcl" package="R1206" value="1k" x="26.3525" y="26.3525" smashed="yes" rot="R270">
 <attribute name="NAME" x="23.6225" y="26.6225" size="1.27" layer="25" font="vector" ratio="15" rot="R270"/>
 <attribute name="VALUE" x="23.8125" y="27.6225" size="1.27" layer="27" font="vector" ratio="15" rot="R270"/>
 </element>
-<element name="R10" library="rcl" package="R1206" value="100k" x="40.3225" y="25.7175"/>
-<element name="T1" library="transistor-fet" package="SO08-IRF" value="IRF7306" x="40.3225" y="19.685" rot="R180"/>
+<element name="R10" library="rcl" package="R1206" value="100k" x="40.3225" y="25.7175" smashed="yes">
+<attribute name="NAME" x="39.0525" y="26.9875" size="1.27" layer="25" font="vector" ratio="15"/>
+<attribute name="VALUE" x="39.0525" y="23.1775" size="1.27" layer="27" font="vector" ratio="15"/>
+</element>
+<element name="T1" library="transistor-fet" package="SO08-IRF" value="IRF7306" x="40.3225" y="19.685" smashed="yes" rot="R180">
+<attribute name="NAME" x="43.18" y="19.685" size="1.27" layer="25" font="vector" ratio="15" rot="R270" align="bottom-center"/>
+<attribute name="VALUE" x="37.465" y="19.685" size="1.27" layer="27" font="vector" ratio="15" rot="R270" align="top-center"/>
+</element>
 <element name="C10" library="rcl" package="E2-5" value="22u/25V" x="48.625" y="32.0675" smashed="yes">
 <attribute name="NAME" x="47.927" y="35.3615" size="1.27" layer="25" ratio="10"/>
 <attribute name="VALUE" x="45.339" y="34.0195" size="1.27" layer="27" ratio="10"/>
 </element>
-<element name="J5" library="con-malina" package="WEBP6-6_SPEC2" value="WEBP6" x="44.7675" y="5.08" populate="no" smashed="yes">
+<element name="J5" library="con-malina" package="WEBP6-6_SPEC2" value="WEBP6" x="44.7675" y="5.08" smashed="yes">
 <attribute name="NAME" x="44.4015" y="3.389" size="1.778" layer="25" rot="R90"/>
 </element>
-<element name="J6" library="con-malina" package="WEBP6-6_SPEC2" value="WEBP6" x="31.115" y="5.08" populate="no" smashed="yes">
+<element name="J6" library="con-malina" package="WEBP6-6_SPEC2" value="WEBP6" x="31.115" y="5.08" smashed="yes">
 <attribute name="NAME" x="30.249" y="3.389" size="1.778" layer="25" rot="R90"/>
 </element>
@@
 <attribute name="NAME" x="58.071" y="20.4065" size="1.778" layer="25" rot="R180"/>
 </element>
-<element name="X2" library="con-malina" package="ARK1550/2_SPEC" value="ARK1550/2_S" x="43.18" y="37.1475" populate="no" smashed="yes" rot="R180"/>
+<element name="X2" library="con-malina" package="ARK1550/2_SPEC" value="ARK1550/2_S" x="43.18" y="37.1475" smashed="yes" rot="R180"/>
 <element name="LED5" library="led" package="LED3MM" value="RED 2mA" x="54.9275" y="12.065" smashed="yes" rot="MR270">
 <attribute name="NAME" x="58.3875" y="12.065" size="1.27" layer="26" ratio="15" rot="MR270" align="bottom-center"/>
 <attribute name="VALUE" x="58.7375" y="12.065" size="1.27" layer="28" ratio="15" rot="MR270" align="bottom-center"/>
 </element>
-<element name="R11" library="rcl" package="R1206" value="10k" x="50.565" y="14.2475" smashed="yes" rot="MR0">
+<element name="R11" library="rcl" package="R1206" value="2k2" x="50.565" y="14.2475" smashed="yes" rot="MR0">
 <attribute name="NAME" x="51.835" y="15.5175" size="1.27" layer="26" font="vector" ratio="15" rot="MR0"/>
 <attribute name="VALUE" x="52.335" y="15.7075" size="1.27" layer="28" font="vector" ratio="15" rot="MR0"/>
@@
 </signal>
 </signals>
+<mfgpreviewcolors>
+<mfgpreviewcolor name="soldermaskcolor" color="0xC8008000"/>
+<mfgpreviewcolor name="silkscreencolor" color="0xFFFEFEFE"/>
+<mfgpreviewcolor name="backgroundcolor" color="0xFF282828"/>
+<mfgpreviewcolor name="coppercolor" color="0xFFFFBF00"/>
+<mfgpreviewcolor name="substratecolor" color="0xFF786E46"/>
+</mfgpreviewcolors>
 </board>
 </drawing>

Commit message: Set precise MCP's voltage.
Parts:
- IC3: value MCP130T -> MCP130T-3V
Changed lines of the file:
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@@
 <attribute name="VALUE" x="44.76" y="33.17" size="1.27" layer="27" font="vector" ratio="15" rot="R270"/>
 </element>
-<element name="IC3" library="my" package="SOT23" value="MCP130T" x="25.7" y="21.5" smashed="yes" rot="R180">
+<element name="IC3" library="my" package="SOT23" value="MCP130T-3V" x="25.7" y="21.5" smashed="yes" rot="R180">
 <attribute name="NAME" x="31.105" y="22.595" size="1.27" layer="25" font="vector" ratio="15" rot="R180"/>
 <attribute name="VALUE" x="29.175" y="16.895" size="1.27" layer="27" font="vector" ratio="15" rot="R90"/>

Commit message: Minor board tweaks.
Routing:
- net GND: track 1.46 -> 0.00 mm, vias 1 -> 4
- net +12V: track 29.9 -> 28.8 mm
