File: uLI-05/uLI-05.kicad_sch (KiCad schematic)
At the start: 54 parts, among them J1 STL1550, J2 USB_B, J3 RJ25, J4 RJ25, J5 PROG, Q1 IRF7306, U1 LM78M05_TO252, U2 PC817, U3 PC817, U4 PIC18F14K50-EP, U5 ADM2483xRW, U6 USBLC6-2SC6, Y1 12MHz

Commit message: F1, F2, F3: add JLCPCB_IGNORE.
Parts:
- F1, F2, F3: JLCPCB_IGNORE (none) -> true
Changed lines of the file:
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@@
       (effects (font (size 1.27 1.27)) (justify left))
+    )
+    (property "JLCPCB_IGNORE" "true" (at 258.445 97.155 0)
+      (effects (font (size 1.27 1.27)) hide)
     )
     (pin "1")
@@
       (effects (font (size 1.27 1.27)) (justify right))
     )
+    (property "JLCPCB_IGNORE" "true" (at 32.385 53.975 0)
+      (effects (font (size 1.27 1.27)) hide)
+    )
     (pin "2")
     (pin "1")
@@
       (effects (font (size 1.27 1.27)))
     )
-    (pin "1")
+    (property "JLCPCB_IGNORE" "true" (at 269.24 32.385 0)
+      (effects (font (size 1.27 1.27)) hide)
+    )
+    (pin "1")

Commit message: D1, D2: add JLCPCB_CORRECTION.
Parts:
- D1, D2: JLCPCB_CORRECTION (none) -> 0;0;180
Changed lines of the file:
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@@
+      (effects (font (size 1.27 1.27)) hide)
+    )
+    (property "JLCPCB_CORRECTION" "0;0;180" (at 246.38 32.385 0)
       (effects (font (size 1.27 1.27)) hide)
     )
@@
       (effects (font (size 1.27 1.27)) hide)
     )
+    (property "JLCPCB_CORRECTION" "0;0;180" (at 260.35 32.385 0)
+      (effects (font (size 1.27 1.27)) hide)
+    )
